File: kicad/timer-board.kicad_pcb (KiCad board)
At the start: 2 copper layers, 15 parts, among them J1 Conn_01x05_Female, SW1 SW_SPST, SW2 SW_SPDT, U1 NE555DR, U2 SN74HC00DR

Commit message: Rework
Parts:
- added J2: Conn_Data, Connector_PinHeader_2.54mm:PinHeader_2x01_P2.54mm_Vertical, F.Cu at (359.9, 121.4)
- J1: value Conn_01x05_Female -> Conn_PWR; footprint Connector_PinHeader_1.00mm:PinHeader_1x05_P1.00mm_Vertical -> Connector_PinHeader_2.54mm:PinHeader_2x01_P2.54mm_Vertical
- U1: footprint NE555DR:SOIC127P600X175-8N -> SOIC127P600X175-8N
- U2: footprint SN74HC00DR:SOIC127P600X175-14N -> SOIC127P600X175-14N
- moved RV1 179.9 mm to (320.1, 118.7)
- moved R4 168.8 mm to (345.9, 113.0), turned to 180 degrees
- moved SW1 168.1 mm to (308.4, 113.3), turned to 270 degrees
- moved U1 167.9 mm to (335.5, 117.3)
- moved U2 165.5 mm to (348.5, 123.0)
- moved D1 165.3 mm to (354.0, 120.7), turned to 0 degrees
- moved R5 165.1 mm to (354.1, 122.7), turned to 0 degrees
- moved C3 164.2 mm to (335.5, 113.5), turned to 180 degrees
- moved SW2 163.7 mm to (325.1, 108.2), turned to 0 degrees
- moved C1 163.1 mm to (328.9, 121.2), turned to 90 degrees
- moved C2 162.2 mm to (335.5, 112.3)
- moved J1 156.6 mm to (359.9, 106.7), turned to 270 degrees
- moved R2 156.6 mm to (328.9, 116.8), turned to 270 degrees
- moved R3 155.2 mm to (328.9, 119.1), turned to 270 degrees
- moved R1 145.4 mm to (316.0, 114.2), turned to 270 degrees
Connections:
- net 5V renamed +5V
- R4 pad 2: Net-(J1-Pad5) -> Net-(J2-Pad2)
- U2 pad 2: Net-(J1-Pad5) -> Net-(J2-Pad2)
- U2 pad 3: Net-(J1-Pad4) -> Net-(J2-Pad1)
- U2 pad 4: Net-(J1-Pad4) -> Net-(J2-Pad1)
Routing:
- net +5V: track 132.7 -> 0.00 mm
- net GND: track 87.0 -> 0.00 mm, vias 2 -> 0
- net Net-(R2-Pad2): track 78.7 -> 0.00 mm
- net Net-(J1-Pad5): track 56.3 -> 0.00 mm, vias 1 -> 0
- net Net-(C1-Pad1): track 43.7 -> 0.00 mm, vias 1 -> 0
- net Net-(R3-Pad1): track 38.7 -> 0.00 mm
- net Net-(R1-Pad1): track 33.6 -> 0.00 mm
- net Net-(D1-Pad2): track 32.1 -> 0.00 mm
- net Net-(U1-Pad3): track 29.7 -> 0.00 mm
- net Net-(J1-Pad4): track 26.3 -> 0.00 mm, vias 1 -> 0
- net Net-(C3-Pad1): track 11.1 -> 0.00 mm, vias 2 -> 0
- net Net-(D1-Pad1): track 2.66 -> 0.00 mm
- added copper zone on F.Cu, net GND
Other:
- board outline added: 61 x 27.9 mm

Commit message: tracks with errors
Parts:
- moved R5 3.30 mm to (357.1, 121.4)
- moved D1 0.92 mm to (354.6, 121.4), turned to 180 degrees
Routing:
- net Net-(C1-Pad1): track 0.00 -> 28.9 mm
- net Net-(J2-Pad2): track 0.00 -> 27.3 mm
- net Net-(J2-Pad1): track 0.00 -> 23.1 mm, vias 0 -> 2
- net Net-(R2-Pad2): track 0.00 -> 18.9 mm
- net Net-(R1-Pad1): track 0.00 -> 16.8 mm
- net Net-(U1-Pad3): track 0.00 -> 14.1 mm
- net +5V: track 0.00 -> 13.4 mm, vias 0 -> 6
- net Net-(D1-Pad2): track 0.00 -> 10.7 mm
- net GND: track 0.00 -> 10.2 mm, vias 0 -> 2
- net Net-(C3-Pad1): track 0.00 -> 10.1 mm
- net Net-(R3-Pad1): track 0.00 -> 8.87 mm
- net Net-(D1-Pad1): track 0.00 -> 1.46 mm
- added copper zone on B.Cu, net +5V
Other:
- net class 5V removed
- net class GND removed

Commit message: Text
Other:
- board text added: "0V"
- board text added: "5V"
- board text added: "AUTO"
- board text added: "CLK"
- board text added: "HLD"
- board text added: "MANU"
- board text added: "Rhobotify Ltd"
- board text added: "Timer V1.0"
Changed lines of the file:
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@@
   (general
     (thickness 1.6)
-    (drawings 4)
+    (drawings 12)
     (tracks 115)
     (zones 0)
@@
     (descr "Through hole straight pin header, 2x01, 2.54mm pitch, double rows")
     (tags "Through hole pin header THT 2x01 2.54mm double row")
-    (fp_text reference J1 (at 1.27 -2.33 90) (layer F.SilkS)
+    (fp_text reference J1 (at 1.27 2.54 180) (layer F.SilkS)
       (effects (font (size 1 1) (thickness 0.15)))
     )
@@
     (descr "Through hole straight pin header, 2x01, 2.54mm pitch, double rows")
     (tags "Through hole pin header THT 2x01 2.54mm double row")
-    (fp_text reference J2 (at 1.27 -2.33 90) (layer F.SilkS)
+    (fp_text reference J2 (at 1.27 2.54 180) (layer F.SilkS)
       (effects (font (size 1 1) (thickness 0.15)))
     )
@@
       (net 14 +5V))
   )
+  (gr_text "Rhobotify Ltd" (at 312.42 125.984) (layer F.SilkS)
+    (effects (font (size 1 1) (thickness 0.15)))
+  )
+  (gr_text "Timer V1.0" (at 344.932 106.426) (layer F.SilkS)
+    (effects (font (size 1 1) (thickness 0.15)))
+  )
+  (gr_text AUTO (at 315.468 118.364) (layer F.SilkS)
+    (effects (font (size 1 1) (thickness 0.15)))
+  )
+  (gr_text MANU (at 315.468 108.204) (layer F.SilkS)
+    (effects (font (size 1 1) (thickness 0.15)))
+  )
+  (gr_text HLD (at 362.966 123.952) (layer F.SilkS)
+    (effects (font (size 1 1) (thickness 0.15)))
+  )
+  (gr_text CLK (at 362.966 121.412) (layer F.SilkS)
+    (effects (font (size 1 1) (thickness 0.15)))
+  )
+  (gr_text 0V (at 362.458 109.22) (layer F.SilkS)
+    (effects (font (size 1 1) (thickness 0.15)))
+  )
+  (gr_text 5V (at 362.458 106.68) (layer F.SilkS)
+    (effects (font (size 1 1) (thickness 0.15)))
+  )
   (gr_line (start 304.8 129.54) (end 304.8 101.6) (layer Edge.Cuts) (width 0.05))

Commit message: More work
Parts:
- added D2: LED - red FV 2V, LED_SMD:LED_0603_1608Metric, F.Cu at (354.6, 119.6)
- added R6: 150, Resistor_SMD:R_0201_0603Metric, F.Cu at (357.1, 119.6)
- R4: value 100K -> 1K
- moved R1 9.16 mm to (325.1, 113.6)
- moved R4 8.10 mm to (352.0, 118.4), turned to 90 degrees
- moved R2 7.97 mm to (333.0, 123.6)
- moved C3 7.11 mm to (335.6, 120.7)
- moved D1 4.57 mm to (354.6, 116.8)
- moved J2 4.57 mm to (359.9, 116.8)
- moved R5 4.57 mm to (357.1, 116.8)
- moved C2 1.78 mm to (335.5, 114.0), turned to 180 degrees
- turned C1 to 270 degrees
Connections:
- J2 pad 1: Net-(J2-Pad1) -> Net-(D1-Pad2)
- J2 pad 2: Net-(J2-Pad2) -> /Hold
- R4 pad 1: +5V -> /Hold
- R4 pad 2: Net-(J2-Pad2) -> GND
- RV1 pad 3: Net-(RV1-Pad3) -> (no net)
- SW2 pad 1: Net-(SW2-Pad1) -> (no net)
- U2 pad 10: GND -> /Hold
- U2 pad 11: Net-(U2-Pad11) -> (no net)
- U2 pad 2: Net-(J2-Pad2) -> /~Hold~
- U2 pad 3: Net-(J2-Pad1) -> Net-(U2-Pad3)
- U2 pad 4: Net-(J2-Pad1) -> Net-(U2-Pad3)
- U2 pad 5: +5V -> Net-(U2-Pad3)
- U2 pad 8: Net-(U2-Pad8) -> /~Hold~
- U2 pad 9: GND -> /Hold
Routing:
- net +5V: track 13.4 -> 88.2 mm, vias 6 -> 2
- net Net-(J2-Pad2): track 27.3 -> 0.00 mm
- net Net-(J2-Pad1): track 23.1 -> 0.00 mm, vias 2 -> 0
- net /~Hold~: track 0.00 -> 17.0 mm
- net /Hold: track 0.00 -> 16.7 mm
- net Net-(D1-Pad2): track 10.7 -> 26.5 mm, vias 0 -> 2
- net Net-(U1-Pad3): track 14.1 -> 26.8 mm, vias 0 -> 2
- net GND: track 10.2 -> 18.8 mm, vias 2 -> 7
- net Net-(C3-Pad1): track 10.1 -> 2.94 mm
- net Net-(C1-Pad1): track 28.9 -> 22.7 mm
- net Net-(R1-Pad1): track 16.8 -> 21.4 mm
- net Net-(R2-Pad2): track 18.9 -> 22.1 mm
- net Net-(U2-Pad3): track 0.00 -> 2.54 mm
- net Net-(D2-Pad1): track 0.00 -> 1.43 mm
- added copper zone on B.Cu, net GND
- removed copper zone on B.Cu, net +5V
- removed copper zone on F.Cu, net GND

Commit message: Fix rules
Other:
- net class Default: clearance 0.2 -> 0.0889
- rule trace_clearance: 0.2 -> 0.0889
- rule trace_min: 0.2 -> 0.0889
Changed lines of the file:
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@@
   (setup
     (last_trace_width 0.25)
-    (trace_clearance 0.2)
+    (trace_clearance 0.0889)
     (zone_clearance 0.508)
     (zone_45_only no)
-    (trace_min 0.2)
+    (trace_min 0.0889)
     (via_size 0.8)
     (via_drill 0.4)
@@
   (net 14 "Net-(U2-Pad3)")
   (net_class Default "This is the default net class."
-    (clearance 0.2)
+    (clearance 0.0889)
     (trace_width 0.25)
     (via_dia 0.8)
