File: kicad/timer-board.kicad_pcb (KiCad board)
At the start: 2 copper layers, 68.6 x 27.9 mm, 19 parts, among them J1 Conn_PWR, J2 Conn_Data, J3 JST Conn, SW1 SW_SPST, SW2 SW_SPDT, U1 NE555DR, U2 SN74HC00DR

Commit message: Version 1.2
Parts:
- SW1: value SW_SPST -> SW_Push_SPDT; footprint mine:snap spst switch -> mine:switch_push_spdt
- SW2: footprint A101SYCQ04:TE_A101SYCQ04 -> mine:switch_toggle_spdt
- moved SW2 7.67 mm to (318.6, 112.3)
Connections:
- SW1 pad 1: +5V -> Net-(R1-Pad1)
- SW1 pad 2: Net-(R1-Pad1) -> +5V
Other:
- board text added: "MAN"
- board text removed: "MANU"
Changed lines of the file:
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@@
     (thickness 1.6)
     (drawings 16)
-    (tracks 134)
+    (tracks 133)
     (zones 0)
     (modules 19)
@@
     (add_net "Net-(U2-Pad3)")
   )
+  (module mine:switch_toggle_spdt (layer F.Cu)
+    (at 318.62 112.268)
+    (fp_text reference SW2 (at 7.6 1) (layer F.SilkS)
+      (effects (font (size 1 1) (thickness 0.15)))
+    )
+    (fp_text value SW_SPDT (at 6.5 -1.1) (layer F.Fab)
+      (effects (font (size 1 1) (thickness 0.15)))
+    )
+    (fp_line (start 0 -8) (end 13 -8) (layer F.SilkS) (width 0.12))
+    (fp_line (start 13 0) (end 13 -8) (layer F.SilkS) (width 0.12))
+    (fp_line (start 0 0) (end 13 0) (layer F.SilkS) (width 0.12))
+    (fp_line (start -0.02 -8) (end -0.02 0) (layer F.SilkS) (width 0.12))
+    (pad 1 thru_hole rect (at 2.125 -4) (size 3.2 3.2) (drill 2.2) (layers *.Cu *.Mask))
+    (pad 2 thru_hole circle (at 6.5 -4) (size 3.2 3.2) (drill oval 1 2.2) (layers *.Cu *.Mask)
+      (net 5 "Net-(R1-Pad1)"))
+    (pad 3 thru_hole circle (at 10.875 -4) (size 3.2 3.2) (drill oval 1 2.2) (layers *.Cu *.Mask)
+      (net 2 "Net-(C1-Pad1)"))
+  )
+  (module mine:switch_push_spdt (layer F.Cu)
+    (at 308.356 115.57 270)
+    (fp_text reference SW1 (at 0 0.5 90) (layer F.SilkS)
+      (effects (font (size 1 1) (thickness 0.15)))
+    )
+    (fp_text value SW_Push_SPDT (at 0 -0.5 90) (layer F.Fab)
+      (effects (font (size 1 1) (thickness 0.15)))
+    )
+    (fp_line (start -5.1 -5.1) (end 7 -10) (layer F.SilkS) (width 0.2))
+    (fp_line (start 7.62 -5.08) (end -7.62 -5.08) (layer F.SilkS) (width 0.12))
+    (fp_line (start 7.62 0) (end 7.62 -5.08) (layer F.SilkS) (width 0.12))
+    (fp_line (start -7.62 0) (end 7.62 0) (layer F.SilkS) (width 0.12))
+    (fp_line (start -7.62 -5.08) (end -7.62 0) (layer F.SilkS) (width 0.12))
+    (pad 2 thru_hole rect (at -5.08 -2.54 270) (size 2.2 2.2) (drill 1.2) (layers *.Cu *.Mask)
+      (net 9 +5V))
+    (pad 3 thru_hole circle (at 0 -2.54 270) (size 2.2 2.2) (drill 1.2) (layers *.Cu *.Mask))
+    (pad 1 thru_hole circle (at 5.08 -2.54 270) (size 2.2 2.2) (drill 1.2) (layers *.Cu *.Mask)
+      (net 5 "Net-(R1-Pad1)"))
+  )
   (module mine:6mm_trimmer (layer F.Cu)
     (at 318.77 118.122)
@@
     )
   )
-  (module "mine:snap spst switch" (layer F.Cu)
-    (at 308.356 115.57 270)
-    (fp_text reference SW1 (at 0 0.5 270) (layer F.SilkS)
-      (effects (font (size 1 1) (thickness 0.15)))
-    )
-    (fp_text value SW_SPST (at 0 -0.5 270) (layer F.Fab)
-      (effects (font (size 1 1) (thickness 0.15)))
-    )
-    (fp_line (start -7.62 -5.08) (end -7.62 0) (layer F.SilkS) (width 0.12))
-    (fp_line (start -7.62 0) (end 7.62 0) (layer F.SilkS) (width 0.12))
-    (fp_line (start 7.62 0) (end 7.62 -5.08) (layer F.SilkS) (width 0.12))
-    (fp_line (start 7.62 -5.08) (end -7.62 -5.08) (layer F.SilkS) (width 0.12))
-    (pad 2 thru_hole circle (at 5.08 -2.54 270) (size 2.2 2.2) (drill 1.2) (layers *.Cu *.Mask)
-      (net 5 "Net-(R1-Pad1)"))
-    (pad X thru_hole circle (at 0 -2.54 270) (size 2.2 2.2) (drill 1.2) (layers *.Cu *.Mask))
-    (pad 1 thru_hole rect (at -5.08 -2.54 270) (size 2.2 2.2) (drill 1.2) (layers *.Cu *.Mask)
-      (net 9 +5V))
-  )
   (module LED_SMD:LED_0603_1608Metric (layer F.Cu)
     (at 352.933 119.507 180)
@@
       (rotate (xyz 0 0 0))
     )
-  )
-  (module A101SYCQ04:TE_A101SYCQ04 (layer F.Cu)
-    (at 325.12 108.204)
-    (fp_text reference SW2 (at -3.75684 -4.71444) (layer F.SilkS)
-      (effects (font (size 1.00001 1.00001) (thickness 0.05)))
-    )
-    (fp_text value SW_SPDT (at -3.12902 4.83747) (layer F.SilkS)
-      (effects (font (size 1.00014 1.00014) (thickness 0.05)))
-    )
-    (fp_line (start -6.35 3.429) (end 6.35 3.429) (layer F.SilkS) (width 0.127))
-    (fp_line (start 6.35 3.429) (end 6.35 -3.429) (layer Eco2.User) (width 0.127))
-    (fp_line (start 6.35 -3.429) (end -6.35 -3.429) (layer F.SilkS) (width 0.127))
-    (fp_line (start -6.35 -3.429) (end -6.35 3.429) (layer Eco2.User) (width 0.127))
-    (fp_line (start -6.6 -3.679) (end 6.6 -3.679) (layer Eco1.User) (width 0.05))
-    (fp_line (start 6.6 -3.679) (end 6.6 3.679) (layer Eco1.User) (width 0.05))
-    (fp_line (start 6.6 3.679) (end -6.6 3.679) (layer Eco1.User) (width 0.05))
-    (fp_line (start -6.6 3.679) (end -6.6 -3.679) (layer Eco1.User) (width 0.05))
-    (fp_circle (center -7.112 -0.001) (end -6.912 -0.001) (layer F.SilkS) (width 0.3))
-    (pad 1 thru_hole rect (at -4.699 0 90) (size 2.7813 2.7813) (drill 1.8542) (layers *.Cu *.Mask))
-    (pad 2 thru_hole circle (at 0 0 90) (size 2.7813 2.7813) (drill 1.8542) (layers *.Cu *.Mask)
-      (net 5 "Net-(R1-Pad1)"))
-    (pad 3 thru_hole circle (at 4.699 0 90) (size 2.7813 2.7813) (drill 1.8542) (layers *.Cu *.Mask)
-      (net 2 "Net-(C1-Pad1)"))
   )
   (module SOIC127P600X175-8N (layer F.Cu)
@@
   (gr_arc (start 307.34 104.14) (end 307.34 101.6) (angle -90) (layer Edge.Cuts) (width 0.05))
   (gr_arc (start 370.84 104.14) (end 373.38 104.14) (angle -90) (layer Edge.Cuts) (width 0.05))
-  (gr_text "Rhobotify Ltd" (at 332.232 127.254) (layer F.SilkS)
+  (gr_text "Rhobotify Ltd" (at 357.886 104.394) (layer F.SilkS)
     (effects (font (size 1 1) (thickness 0.15)))
   )
@@
     (effects (font (size 1 1) (thickness 0.15)))
   )
-  (gr_text AUTO (at 315.468 118.364) (layer F.SilkS)
+  (gr_text AUTO (at 334.264 108.204) (layer F.SilkS)
     (effects (font (size 1 1) (thickness 0.15)))
   )
-  (gr_text MANU (at 315.468 108.204) (layer F.SilkS)
+  (gr_text MAN (at 316.484 108.204) (layer F.SilkS)
     (effects (font (size 1 1) (thickness 0.15)))
   )
@@
   (segment (start 336.7572 117.983) (end 335.4872 116.713) (width 0.25) (layer F.Cu) (net 2))
   (segment (start 337.9978 117.983) (end 336.7572 117.983) (width 0.25) (layer F.Cu) (net 2))
-  (segment (start 329.819 110.170676) (end 329.819 108.204) (width 0.25) (layer F.Cu) (net 2))
-  (segment (start 329.819 114.7024) (end 329.819 110.170676) (width 0.25) (layer F.Cu) (net 2))
-  (segment (start 331.8296 116.713) (end 329.819 114.7024) (width 0.25) (layer F.Cu) (net 2))
-  (segment (start 333.0702 116.713) (end 331.8296 116.713) (width 0.25) (layer F.Cu) (net 2))
   (segment (start 328.93 121.8945) (end 328.93 120.4215) (width 0.25) (layer F.Cu) (net 2))
   (segment (start 332.6385 116.713) (end 333.0702 116.713) (width 0.25) (layer F.Cu) (net 2))
   (segment (start 328.93 120.4215) (end 332.6385 116.713) (width 0.25) (layer F.Cu) (net 2))
+  (segment (start 329.495 114.3784) (end 329.495 108.268) (width 0.25) (layer F.Cu) (net 2))
+  (segment (start 333.0702 116.713) (end 331.8296 116.713) (width 0.25) (layer F.Cu) (net 2))
+  (segment (start 331.8296 116.713) (end 329.495 114.3784) (width 0.25) (layer F.Cu) (net 2))
   (segment (start 337.9978 119.253) (end 337.9978 120.0404) (width 0.25) (layer F.Cu) (net 3))
   (segment (start 337.9978 120.0404) (end 337.312 120.7262) (width 0.25) (layer F.Cu) (net 3))
